Commit message: 12_14

File: sentry_description/urdf/sentry_description.urdf (robot description, URDF)
Before this commit: robot sentry_description, 11 links, 10 joints
Joints:
- joint imu_joint: origin xyz=0 0 0 rpy=3.14 0 0 -> xyz=0 0 0 rpy=0 0 0
- joint lidar_joint: origin xyz=0 0 0.316500899999999 rpy=-3.14159265358979 0 0 -> xyz=0 0 0.316500899999999 rpy=0 0 0

Commit message: 1_10_2

File: sentry_description/urdf/sentry_description.urdf (robot description, URDF)
Before this commit: robot sentry_description, 11 links, 10 joints
Joints:
- joint lidar_joint: origin xyz=0 0 0.316500899999999 rpy=0 0 0 -> xyz=0 0 0.40806 rpy=0 0 0.78539815

Commit message: 1_1145度第一版

File: sentry_description/urdf/sentry_description.urdf (robot description, URDF)
Before this commit: robot sentry_description, 11 links, 10 joints
Joints:
- joint lidar_joint: origin xyz=0 0 0.40806 rpy=0 0 0.78539815 -> xyz=0 0 0.40806 rpy=0 0.7853981633974483 0

Commit message: 1_13_usb转can第二代

File: sentry_description/urdf/sentry_description.urdf (robot description, URDF)
Before this commit: robot sentry_description, 11 links, 10 joints
Joints:
- joint imu_joint: origin xyz=0 0 0 rpy=0 0 0 -> xyz=0 0 0 rpy=-0.7853981633974483 0 0 
- joint lidar_joint: origin xyz=0 0 0.40806 rpy=0 0.7853981633974483 0 -> xyz=0 0 0.40806 rpy=-0.7853981633974483 0 0

Commit message: 准备加入pointlio

File: sentry_description/urdf/sentry_description.urdf (robot description, URDF)
Before this commit: robot sentry_description, 11 links, 10 joints
Joints:
- joint imu_joint: origin xyz=0 0 0 rpy=-0.7853981633974483 0 0  -> xyz=0 0 0 rpy=0  0 0 
- joint lidar_joint: origin xyz=0 0 0.40806 rpy=-0.7853981633974483 0 0 -> xyz=0 0 0.40806 rpy=-0.837758  0.017453 0

Commit message: 12——23

File: sentry_description/urdf/sentry_description.urdf (robot description, URDF)
Before this commit: robot sentry_description, 11 links, 10 joints
Joints:
- joint lidar_joint: origin xyz=0 0 0.40806 rpy=-0.837758  0.017453 0 -> xyz=0 0 0.40806 rpy=-0  0 0

Commit message: 改了云台解算，试图加入新仿真建模

File: sentry_description/urdf/sentry_description.urdf (robot description, URDF)
Before this commit: robot sentry_description, 11 links, 10 joints
Joints:
- joint lidar_joint: origin xyz=0 0 0.40806 rpy=-0  0 0 -> xyz=-0.07472 0.15378 0.40806 rpy=0 0 0

Commit message: 第一版本雷达（单雷达）除了裁判系统can通讯全部完成

File: sentry_description/urdf/sentry_description.urdf (robot description, URDF)
Before this commit: robot sentry_description, 11 links, 10 joints
Joints:
- joint lidar_joint: origin xyz=-0.07472 0.15378 0.40806 rpy=0 0 0 -> xyz=-0.11472 0.16078 0.40806 rpy=0 0 0

Commit message: 2——28

File: sentry_description/urdf/sentry_description.urdf (robot description, URDF)
Before this commit: robot sentry_description, 11 links, 10 joints
Joints:
- joint lidar_joint: origin xyz=-0.11472 0.16078 0.40806 rpy=0 0 0 -> xyz=-0.11472 0.16078 0.0 rpy=0 0 0

Commit message: 444

File: sentry_description/urdf/sentry_description.urdf (robot description, URDF)
Before this commit: robot sentry_description, 11 links, 10 joints
Joints:
- joint lidar_joint: origin xyz=-0.11472 0.16078 0.40806 rpy=0 0 0 -> xyz=-0.11472 0.16078 0.00000 rpy=0 0 0

Commit message: 云台解算出问题

File: sentry_description/urdf/sentry_description.urdf (robot description, URDF)
Before this commit: robot sentry_description, 11 links, 10 joints
Joints:
- joint lidar_joint: origin xyz=-0.11472 0.16078 0.00000 rpy=0 0 0 -> xyz=-0.11472 0.14578 0.00000 rpy=0 0 0
